File: Hardware/Colorimetry-Boards/LEDCarrier.sch (KiCad schematic (older format))
At the start: 22 parts, among them IC1 ATTINY48-M, P1 CONN_01X04, P2 CONN_01X04, P3 CONN_02X05, P6 CONN_02X03, Q1 2N7002P, Q2 2N7002P, Q3 NTR4003N, U1 AP2114H-3.3TRG1, U2 VEML6040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

Commit message: Renaming and finished boards
Also reworked color sensor board
Parts:
- removed P3: CONN_02X05, RST-Footprints:PAD-2x5, symbol CONN_02X05
- P4, P5: renamed from P?; footprint (none) -> Pin_Headers:Pin_Header_Straight_1x04
Connections:
- wire segments 100 -> 68
- no-connect marks 14 -> 22
Other:
- note removed: "GPIO\n"
Changed lines of the file:
@@
 Text GLabel 4500 4800 0    60   Input ~ 0
-VCC
-$Comp
-L CONN_02X05 P3
-U 1 1 563F706C
-P 7450 4800
-F 0 "P3" H 7450 5100 50  0000 C CNN
-F 1 "CONN_02X05" H 7450 4500 50  0000 C CNN
-F 2 "RST-Footprints:PAD-2x5" H 7450 3600 60  0001 C CNN
-F 3 "" H 7450 3600 60  0000 C CNN
-F 4 "N/P" H 7450 4800 60  0001 C CNN "Digikey PN"
-	1    7450 4800
-	0    1    1    0
-$EndComp
-Text GLabel 7650 5050 3    60   Input ~ 0
-GND
-Text GLabel 7650 4550 1    60   Input ~ 0
 VCC
 Text GLabel 6600 2300 2    60   Input ~ 0
 LEDC
 $Comp
-L GND #PWR01
+L GND #PWR2
 U 1 1 563F7BE2
 P 8000 2700
-F 0 "#PWR01" H 8000 2450 50  0001 C CNN
+F 0 "#PWR2" H 8000 2450 50  0001 C CNN
 F 1 "GND" H 8000 2550 50  0000 C CNN
 F 2 "" H 8000 2700 60  0000 C CNN
@@
 $EndComp
 $Comp
-L +5V #PWR02
+L +5V #PWR1
 U 1 1 563F7BFD
 P 8000 2400
-F 0 "#PWR02" H 8000 2250 50  0001 C CNN
+F 0 "#PWR1" H 8000 2250 50  0001 C CNN
 F 1 "+5V" H 8000 2540 50  0000 C CNN
 F 2 "" H 8000 2400 60  0000 C CNN
@@
 Connection ~ 6950 3500
 Wire Wire Line
-	6600 4750 7000 4750
-Wire Wire Line
-	7000 4750 7000 4500
-Wire Wire Line
-	7000 4500 7250 4500
-Wire Wire Line
-	7250 4500 7250 4550
-Wire Wire Line
-	6600 4650 6950 4650
-Wire Wire Line
-	6950 4650 6950 4450
-Wire Wire Line
-	6950 4450 7350 4450
-Wire Wire Line
-	7350 4450 7350 4550
-Wire Wire Line
-	7450 4550 7450 4400
-Wire Wire Line
-	7450 4400 6900 4400
-Wire Wire Line
-	6900 4400 6900 4550
-Wire Wire Line
-	6900 4550 6600 4550
-Wire Wire Line
-	6600 4450 6850 4450
-Wire Wire Line
-	6850 4450 6850 4350
-Wire Wire Line
-	6850 4350 7550 4350
-Wire Wire Line
-	7550 4350 7550 4550
-Wire Wire Line
-	6600 4850 7000 4850
-Wire Wire Line
-	7000 4850 7000 5100
-Wire Wire Line
-	7000 5100 7250 5100
-Wire Wire Line
-	7250 5100 7250 5050
-Wire Wire Line
-	7350 5050 7350 5150
-Wire Wire Line
-	7350 5150 6950 5150
-Wire Wire Line
-	6950 5150 6950 4950
-Wire Wire Line
-	6950 4950 6600 4950
-Wire Wire Line
-	6600 5050 6900 5050
-Wire Wire Line
-	6900 5050 6900 5200
-Wire Wire Line
-	6900 5200 7450 5200
-Wire Wire Line
-	7450 5200 7450 5050
-Wire Wire Line
-	7550 5050 7550 5250
-Wire Wire Line
-	7550 5250 6850 5250
-Wire Wire Line
-	6850 5250 6850 5150
-Wire Wire Line
-	6850 5150 6600 5150
-Wire Wire Line
 	4500 5100 4650 5100
 Wire Wire Line
@@
 $EndComp
 Wire Wire Line
-	1650 4250 3250 4250
-Wire Wire Line
 	3250 4250 3250 4200
-Connection ~ 1650 4250
 Wire Wire Line
 	3250 3700 3250 3800
@@
 Wire Notes Line
 	4150 2050 4150 5400
-Text Notes 7350 4850 0    59   ~ 0
-GPIO\n
 Text Notes 8400 2300 0    59   ~ 0
 (Because an LED on a board\n would be too easy)
@@
 GND
 Wire Wire Line
-	7650 4200 6600 4200
+	6600 4200 7650 4200
 Wire Wire Line
 	7550 4200 7550 4150
@@
 $EndComp
 Text GLabel 7550 3900 1    60   Input ~ 0
-GND
+VCC
 Wire Wire Line
 	7550 3900 7550 3950
@@
 10 42 08 21 84 10 42 08 21 84 10 42 08 21 84 10 42 08 21 84 10 42 08 21 84 10 42 08 21 84 10 42
 08 21 84 10 42 08 21 84 10 42 08 21 84 10 42 08 21 84 10 42 08 21 84 10 42 08 21 84 10 42 08 21
-84 10 42 08 E1 FF DC FF 00 10 1D 96 BE 6F 24 74 FB 00 00 00 00 49 45 4E 44 AE 42 60 82 99
+84 10 42 08 E1 FF DC FF 00 10 1D 96 BE 6F 24 74 FB 00 00 00 00 49 45 4E 44 AE 42 60 82 35
 EndData
 $EndBitmap
 $Comp
-L CONN_01X04 P?
+L CONN_01X04 P4
 U 1 1 56419BC0
 P 1700 2900
-F 0 "P?" H 1700 3150 50  0000 C CNN
+F 0 "P4" H 1700 3150 50  0000 C CNN
 F 1 "CONN_01X04" V 1800 2900 50  0000 C CNN
-F 2 "" H 1700 2900 60  0000 C CNN
+F 2 "Pin_Headers:Pin_Header_Straight_1x04" H 1700 2900 60  0001 C CNN
 F 3 "" H 1700 2900 60  0000 C CNN
 	1    1700 2900
@@
 $EndComp
 $Comp
-L CONN_01X04 P?
+L CONN_01X04 P5
 U 1 1 56419C1C
 P 1700 4500
-F 0 "P?" H 1700 4750 50  0000 C CNN
+F 0 "P5" H 1700 4750 50  0000 C CNN
 F 1 "CONN_01X04" V 1800 4500 50  0000 C CNN
-F 2 "" H 1700 4500 60  0000 C CNN
+F 2 "Pin_Headers:Pin_Header_Straight_1x04" H 1700 4500 60  0001 C CNN
 F 3 "" H 1700 4500 60  0000 C CNN
 	1    1700 4500
 	0    -1   1    0
 $EndComp
+Wire Wire Line
+	3250 4250 1750 4250
+Connection ~ 1750 4250
+NoConn ~ 6600 4450
+NoConn ~ 6600 4550
+NoConn ~ 6600 4650
+NoConn ~ 6600 4750
+NoConn ~ 6600 4850
+NoConn ~ 6600 4950
+NoConn ~ 6600 5050
+NoConn ~ 6600 5150
 $EndSCHEMATC

Commit message: Finished Hardware
Now we wait for it all to arrive
Parts:
- D1: Digikey PN (none) -> XREWHT-L1-0000-006E5CT-ND
- P1, P2, P4, P5: Digikey PN (none) -> A1927-ND
- P6: Digikey PN (none) -> S9015E-03-ND
- Q3: Digikey PN (none) -> NTR4003NT1GOSCT-ND
- R1, R2: Digikey PN RHM4.7KDCT-ND -> 311-4.7KGRCT-ND
- R3, R4: Digikey PN (none) -> 311-2.2KGRCT-ND
- R5, R6: Digikey PN (none) -> 311-10KGRCT-ND
Changed lines of the file:
@@
 F 2 "Pin_Headers:Pin_Header_Straight_1x04" H 8200 2550 60  0001 C CNN
 F 3 "" H 8200 2550 60  0000 C CNN
+F 4 "A1927-ND" H 8200 2550 60  0001 C CNN "Digikey PN"
 	1    8200 2550
 	1    0    0    -1
@@
 F 2 "Pin_Headers:Pin_Header_Straight_1x04" H 8200 3100 60  0001 C CNN
 F 3 "" H 8200 3100 60  0000 C CNN
+F 4 "A1927-ND" H 8200 3100 60  0001 C CNN "Digikey PN"
 	1    8200 3100
 	1    0    0    -1
@@
 F 2 "Resistors_SMD:R_0603" V 6680 3750 30  0001 C CNN
 F 3 "" H 6750 3750 30  0000 C CNN
-F 4 "RHM4.7KDCT-ND" H 6750 3750 60  0001 C CNN "Digikey PN"
+F 4 "311-4.7KGRCT-ND" H 6750 3750 60  0001 C CNN "Digikey PN"
 	1    6750 3750
 	1    0    0    -1
@@
 F 2 "Resistors_SMD:R_0603" V 6880 3750 30  0001 C CNN
 F 3 "" H 6950 3750 30  0000 C CNN
-F 4 "RHM4.7KDCT-ND" H 6950 3750 60  0001 C CNN "Digikey PN"
+F 4 "311-4.7KGRCT-ND" H 6950 3750 60  0001 C CNN "Digikey PN"
 	1    6950 3750
 	1    0    0    -1
@@
 F 2 "Resistors_SMD:R_0603" H 2100 3450 60  0001 C CNN
 F 3 "" H 2100 3450 60  0000 C CNN
+F 4 "311-2.2KGRCT-ND" H 2100 3450 60  0001 C CNN "Digikey PN"
 	1    2100 3450
 	1    0    0    -1
@@
 F 2 "Resistors_SMD:R_0603" H 3400 3750 60  0001 C CNN
 F 3 "" H 3400 3750 60  0000 C CNN
+F 4 "311-2.2KGRCT-ND" H 3400 3750 60  0001 C CNN "Digikey PN"
 	1    3400 3750
 	0    1    1    0
@@
 F 2 "RST-Footprints:XR-E-2-SMD" H 9200 3700 59  0001 C CNN
 F 3 "" H 9200 3700 59  0000 C CNN
+F 4 "XREWHT-L1-0000-006E5CT-ND" H 9200 3700 60  0001 C CNN "Digikey PN"
 	1    9200 3700
 	1    0    0    -1
@@
 F 2 "Housings_SOT-23_SOT-143_TSOT-6:SOT-23" H 9400 4100 60  0001 C CNN
 F 3 "" H 9400 4100 60  0000 C CNN
+F 4 "NTR4003NT1GOSCT-ND" H 9400 4100 60  0001 C CNN "Digikey PN"
 	1    9400 4100
 	1    0    0    -1
@@
 F 2 "Resistors_SMD:R_0603" H 9000 4250 60  0001 C CNN
 F 3 "" H 9000 4250 60  0000 C CNN
+F 4 "311-10KGRCT-ND" H 9000 4250 60  0001 C CNN "Digikey PN"
 	1    9000 4250
 	1    0    0    -1
@@
 F 2 "Pin_Headers:Pin_Header_Straight_2x03" H 9100 1700 60  0001 C CNN
 F 3 "" H 9100 1700 60  0000 C CNN
+F 4 "S9015E-03-ND" H 9100 2900 60  0001 C CNN "Digikey PN"
 	1    9100 2900
 	1    0    0    -1
@@
 F 2 "Resistors_SMD:R_0603" H 7550 4050 60  0001 C CNN
 F 3 "" H 7550 4050 60  0000 C CNN
+F 4 "311-10KGRCT-ND" H 7550 4050 60  0001 C CNN "Digikey PN"
 	1    7550 4050
 	1    0    0    -1
@@
 10 42 08 21 84 10 42 08 21 84 10 42 08 21 84 10 42 08 21 84 10 42 08 21 84 10 42 08 21 84 10 42
 08 21 84 10 42 08 21 84 10 42 08 21 84 10 42 08 21 84 10 42 08 21 84 10 42 08 21 84 10 42 08 21
-84 10 42 08 E1 FF DC FF 00 10 1D 96 BE 6F 24 74 FB 00 00 00 00 49 45 4E 44 AE 42 60 82 35
+84 10 42 08 E1 FF DC FF 00 10 1D 96 BE 6F 24 74 FB 00 00 00 00 49 45 4E 44 AE 42 60 82 DB
 EndData
 $EndBitmap
@@
 F 2 "Pin_Headers:Pin_Header_Straight_1x04" H 1700 2900 60  0001 C CNN
 F 3 "" H 1700 2900 60  0000 C CNN
+F 4 "A1927-ND" H 1700 2900 60  0001 C CNN "Digikey PN"
 	1    1700 2900
 	0    -1   -1   0
@@
 F 2 "Pin_Headers:Pin_Header_Straight_1x04" H 1700 4500 60  0001 C CNN
 F 3 "" H 1700 4500 60  0000 C CNN
+F 4 "A1927-ND" H 1700 4500 60  0001 C CNN "Digikey PN"
 	1    1700 4500
 	0    -1   1    0
